File: Hardware/GX4000-SRAM.kicad_pcb (KiCad board)
At the start: 4 copper layers, 10.2 x 52.1 mm, 11 parts, among them IC10 TMS4464, IC11 TMS4464, U1 IS61C1024AL-12HLI, U2 74HCT573, U3 74LVC1G32, U4 74LVC1G08

Commit message: Update Kicad version to 8
- Update Kicad version format
- Update Footprint
- Add JLCPCB component reference
- Add BOM in description
Parts:
- U2: value 74HCT573 -> SN74HCT573PWR
Connections:
- R1 pad 1: /~{CAS1} -> VCC
- R1 pad 2: VCC -> /~{CAS1}
